File: pcb/skibidi-usb-mux.kicad_pcb (KiCad board)
At the start: 2 copper layers, 75 x 35 mm, 33 parts, among them J1 USB_C_Receptacle_USB2.0_14P, J2 USB_C_Receptacle_USB2.0_14P, J3 USB_C_Receptacle_USB2.0_14P, J4 USB_A, J5 USB_A, J6 USB_A, SW1 PS-5850A-6PL, U1 FSUSB42MUX, U2 CH334P, U3 USBLC6-2SC6, U4 USBLC6-2SC6, U5 USBLC6-2SC6, U6 USBLC6-2SC6, U7 USBLC6-2SC6, U8 USBLC6-2SC6, U9 CH217A

Commit message: add more mentions and art
Other:
- board text added: "Kate"
- board text added: "Tanishq Goyal"
- board text added: "dodge1"
- board text added: "parking_turkeys"
- board text added: "shades"
- board text removed: "Tanuki"
